File: PSU_+12V-12V+5V.kicad_pcb (KiCad board)
At the start: 2 copper layers, 97.2 x 102.2 mm, 61 parts, among them J1 PSU12a, J2 PSU12b, J3 PSU5, J4 230V, Q1 BC557, Q2 BC557, Q3 BC547, Q4 BC547, U1 LM317L, U2 LM317L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

Commit message: Put some nets
Connections:
- net /12Va renamed /OUT12P
- net /12Vb renamed /OUT12N
- net /5Vc renamed /OUT5V
- net Net-(C10-Pad1) renamed /UNR12N
- net Net-(C11-Pad1) renamed /ADJ12P
- net Net-(C12-Pad1) renamed /ADJ12N
- net Net-(C15-Pad1) renamed /ADJ5V
- net Net-(C3-Pad1) renamed /IN12P
- net Net-(C4-Pad1) renamed /IN12N
- net Net-(C5-Pad1) renamed /CAPMULN
- net Net-(C7-Pad1) renamed /CAPMULP
- net Net-(C8-Pad1) renamed /INP5V
- net Net-(C9-Pad1) renamed /UNR12P

Commit message: Changed some values
Parts:
- C13, C14: value 1µ -> 10µ
- R12, R14: value 33k -> 1k8
- R15: value 100 -> 330
- R16: value 560 -> 330
- R6, R9: value 39k -> 100k
Changed lines of the file:
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@@
       (effects (font (size 1 1) (thickness 0.15)))
     )
-    (fp_text value "1µ" (at 1.25 3.75 90) (layer "F.Fab")
+    (fp_text value "10µ" (at 1.25 3.75 90) (layer "F.Fab")
       (effects (font (size 1 1) (thickness 0.15)))
     )
@@
       (effects (font (size 1 1) (thickness 0.15)))
     )
-    (fp_text value "1µ" (at 1.25 3.75 90) (layer "F.Fab")
+    (fp_text value "10µ" (at 1.25 3.75 90) (layer "F.Fab")
       (effects (font (size 1 1) (thickness 0.15)))
     )
@@
       (effects (font (size 1 1) (thickness 0.15)) (justify mirror))
     )
-    (fp_text value "100" (at 0 -1.82 90) (layer "B.Fab")
+    (fp_text value "330" (at 0 -1.82 90) (layer "B.Fab")
       (effects (font (size 1 1) (thickness 0.15)) (justify mirror))
     )
@@
       (effects (font (size 1 1) (thickness 0.15)) (justify mirror))
     )
-    (fp_text value "39k" (at 0 -1.82 -270) (layer "B.Fab")
+    (fp_text value "100k" (at 0 -1.82 -270) (layer "B.Fab")
       (effects (font (size 1 1) (thickness 0.15)) (justify mirror))
     )
@@
       (effects (font (size 1 1) (thickness 0.15)) (justify mirror))
     )
-    (fp_text value "560" (at 0 -1.82) (layer "B.Fab")
+    (fp_text value "330" (at 0 -1.82) (layer "B.Fab")
       (effects (font (size 1 1) (thickness 0.15)) (justify mirror))
     )
@@
       (effects (font (size 1 1) (thickness 0.15)) (justify mirror))
     )
-    (fp_text value "33k" (at 0 -1.82 90) (layer "B.Fab")
+    (fp_text value "1k8" (at 0 -1.82 90) (layer "B.Fab")
       (effects (font (size 1 1) (thickness 0.15)) (justify mirror))
     )
@@
       (effects (font (size 1 1) (thickness 0.15)) (justify mirror))
     )
-    (fp_text value "33k" (at 0 -1.82 90) (layer "B.Fab")
+    (fp_text value "1k8" (at 0 -1.82 90) (layer "B.Fab")
       (effects (font (size 1 1) (thickness 0.15)) (justify mirror))
     )
@@
       (effects (font (size 1 1) (thickness 0.15)) (justify mirror))
     )
-    (fp_text value "39k" (at 0 -1.82 -270) (layer "B.Fab")
+    (fp_text value "100k" (at 0 -1.82 -270) (layer "B.Fab")
       (effects (font (size 1 1) (thickness 0.15)) (justify mirror))
     )
